File: Schematics/lightbox/lightbox.kicad_sch (KiCad schematic)
At the start: 35 parts, among them J1 Screw_Terminal_01x04, J2 Conn_01x11_Female, J3 Conn_01x07_Female, J4 Conn_02x03_Odd_Even, Q1 IRF740, Q2 IRF740, SW1 SW_Push_-, SW2 SW_Push_Reset, SW3 SW_Push_+, SW4 SW_Push_START, SW5 SW_SP3T, U1 74AHCT595, U2 74HC595, U3 ATtiny85-20P, U4 LM317_TO-220

Commit message: Revert schematics
Parts:
- removed Q?: IRF740, Package_TO_SOT_THT:TO-220-3_Vertical, symbol Transistor_FET:IRF740
Connections:
- net Buzzer: now also BZ1.1 (-)
Other:
- moved on the sheet: BZ1
Changed lines of the file:
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@@
     (stroke (width 0) (type default) (color 0 0 0 0))
   )
-  (wire (pts (xy 210.82 41.91) (xy 207.01 41.91))
+  (wire (pts (xy 214.63 40.64) (xy 210.82 40.64))
     (stroke (width 0) (type default) (color 0 0 0 0))
   )
@@
     (stroke (width 0) (type default) (color 0 0 0 0))
   )
-  (wire (pts (xy 207.01 24.13) (xy 207.01 26.67))
-    (stroke (width 0) (type default) (color 0 0 0 0))
-  )
   (wire (pts (xy 193.04 46.99) (xy 193.04 49.53))
     (stroke (width 0) (type default) (color 0 0 0 0))
@@
     (stroke (width 0) (type default) (color 0 0 0 0))
   )
-  (wire (pts (xy 207.01 41.91) (xy 207.01 44.45))
+  (wire (pts (xy 210.82 40.64) (xy 210.82 43.18))
     (stroke (width 0) (type default) (color 0 0 0 0))
   )
@@
     (stroke (width 0) (type default) (color 0 0 0 0))
   )
-  (wire (pts (xy 207.01 36.83) (xy 210.82 36.83))
+  (wire (pts (xy 210.82 35.56) (xy 214.63 35.56))
     (stroke (width 0) (type default) (color 0 0 0 0))
   )
@@
   )
   (wire (pts (xy 190.5 120.65) (xy 190.5 125.73))
-    (stroke (width 0) (type default) (color 0 0 0 0))
-  )
-  (wire (pts (xy 195.58 31.75) (xy 199.39 31.75))
     (stroke (width 0) (type default) (color 0 0 0 0))
   )
@@
     (effects (font (size 1.27 1.27)) (justify left bottom))
   )
-  (label "Buzzer" (at 195.58 31.75 180)
+  (label "Buzzer" (at 210.82 35.56 180)
     (effects (font (size 1.27 1.27)) (justify right bottom))
   )
@@
     (pin "1")
   )
-  (symbol (lib_id "power:GND") (at 207.01 44.45 0) (mirror y) (unit 1)
-    (in_bom yes) (on_board yes) (fields_autoplaced)
-    (property "Reference" "#PWR021" (id 0) (at 207.01 50.8 0)
-      (effects (font (size 1.27 1.27)) hide)
-    )
-    (property "Value" "GND" (id 1) (at 207.01 49.53 0))
-    (property "Footprint" "" (id 2) (at 207.01 44.45 0)
-      (effects (font (size 1.27 1.27)) hide)
-    )
-    (property "Datasheet" "" (id 3) (at 207.01 44.45 0)
+  (symbol (lib_id "power:GND") (at 210.82 43.18 0) (mirror y) (unit 1)
+    (in_bom yes) (on_board yes) (fields_autoplaced)
+    (property "Reference" "#PWR021" (id 0) (at 210.82 49.53 0)
+      (effects (font (size 1.27 1.27)) hide)
+    )
+    (property "Value" "GND" (id 1) (at 210.82 48.26 0))
+    (property "Footprint" "" (id 2) (at 210.82 43.18 0)
+      (effects (font (size 1.27 1.27)) hide)
+    )
+    (property "Datasheet" "" (id 3) (at 210.82 43.18 0)
       (effects (font (size 1.27 1.27)) hide)
     )
@@
     (pin "1")
   )
-  (symbol (lib_id "Transistor_FET:IRF740") (at 204.47 31.75 0) (unit 1)
-    (in_bom yes) (on_board yes) (fields_autoplaced)
-    (property "Reference" "Q?" (id 0) (at 210.82 30.4799 0)
-      (effects (font (size 1.27 1.27)) (justify left))
-    )
-    (property "Value" "IRF740" (id 1) (at 210.82 33.0199 0)
-      (effects (font (size 1.27 1.27)) (justify left))
-    )
-    (property "Footprint" "Package_TO_SOT_THT:TO-220-3_Vertical" (id 2) (at 210.82 33.655 0)
-      (effects (font (size 1.27 1.27) italic) (justify left) hide)
-    )
-    (property "Datasheet" "http://www.vishay.com/docs/91054/91054.pdf" (id 3) (at 204.47 31.75 0)
-      (effects (font (size 1.27 1.27)) (justify left) hide)
-    )
-    (pin "1")
-    (pin "2")
-    (pin "3")
-  )
   (symbol (lib_id "Device:R") (at 77.4996 100.33 90) (unit 1)
     (in_bom yes) (on_board yes)
@@
     )
     (property "Datasheet" "" (id 3) (at 58.42 115.57 0)
-      (effects (font (size 1.27 1.27)) hide)
-    )
-    (pin "1")
-  )
-  (symbol (lib_id "power:+12V") (at 207.01 24.13 0) (unit 1)
-    (in_bom yes) (on_board yes) (fields_autoplaced)
-    (property "Reference" "#PWR?" (id 0) (at 207.01 27.94 0)
-      (effects (font (size 1.27 1.27)) hide)
-    )
-    (property "Value" "+12V" (id 1) (at 207.01 19.05 0))
-    (property "Footprint" "" (id 2) (at 207.01 24.13 0)
-      (effects (font (size 1.27 1.27)) hide)
-    )
-    (property "Datasheet" "" (id 3) (at 207.01 24.13 0)
       (effects (font (size 1.27 1.27)) hide)
     )
@@
     (pin "1")
   )
-  (symbol (lib_id "Device:Buzzer") (at 213.36 39.37 0) (unit 1)
-    (in_bom yes) (on_board yes) (fields_autoplaced)
-    (property "Reference" "BZ1" (id 0) (at 217.17 38.0999 0)
-      (effects (font (size 1.27 1.27)) (justify left))
-    )
-    (property "Value" "Buzzer" (id 1) (at 217.17 40.6399 0)
-      (effects (font (size 1.27 1.27)) (justify left))
-    )
-    (property "Footprint" "Buzzer_Beeper:MagneticBuzzer_ProSignal_ABI-010-RC" (id 2) (at 212.725 36.83 90)
-      (effects (font (size 1.27 1.27)) hide)
-    )
-    (property "Datasheet" "~" (id 3) (at 212.725 36.83 90)
+  (symbol (lib_id "Device:Buzzer") (at 217.17 38.1 0) (unit 1)
+    (in_bom yes) (on_board yes) (fields_autoplaced)
+    (property "Reference" "BZ1" (id 0) (at 220.98 36.8299 0)
+      (effects (font (size 1.27 1.27)) (justify left))
+    )
+    (property "Value" "Buzzer" (id 1) (at 220.98 39.3699 0)
+      (effects (font (size 1.27 1.27)) (justify left))
+    )
+    (property "Footprint" "Buzzer_Beeper:MagneticBuzzer_ProSignal_ABI-010-RC" (id 2) (at 216.535 35.56 90)
+      (effects (font (size 1.27 1.27)) hide)
+    )
+    (property "Datasheet" "~" (id 3) (at 216.535 35.56 90)
       (effects (font (size 1.27 1.27)) hide)
     )
@@
       (reference "#PWR026") (unit 1) (value "GND") (footprint "")
     )
-    (path "/d4977a6e-b824-4cd7-a8e2-21e160fb5299"
-      (reference "#PWR?") (unit 1) (value "+12V") (footprint "")
-    )
     (path "/f0794752-ceaf-4642-b2ee-df197ea3fe2a"
       (reference "BZ1") (unit 1) (value "Buzzer") (footprint "Buzzer_Beeper:MagneticBuzzer_ProSignal_ABI-010-RC")
@@
       (reference "Q2") (unit 1) (value "IRF740") (footprint "Package_TO_SOT_THT:TO-220-3_Vertical")
     )
-    (path "/9ae2bd2d-a780-4ed7-9b7f-8a10db476ae6"
-      (reference "Q?") (unit 1) (value "IRF740") (footprint "Package_TO_SOT_THT:TO-220-3_Vertical")
-    )
     (path "/524d1d1c-f720-4dd7-b8c7-be1393e3f5f7"

Commit message: Update PCB Layout; Update Regulator design
Parts:
- added R11: (no value), Resistor_THT:R_Axial_DIN0204_L3.6mm_D1.6mm_P5.08mm_Vertical, symbol Device:R
- added R8: 10K, Resistor_THT:R_Axial_DIN0204_L3.6mm_D1.6mm_P5.08mm_Vertical, symbol Device:R
- R12: renamed from R10; value 1K -> (none)
- R13: renamed from R11; value 1.5K -> (none)
- renumbered R9 to R10, R8 to R9
Connections:
- net GND: now also R11.1, R8.1
- net REDLeds: now also R8.2
- net UVLeds: now also J3.1 (Pin_1), R11.2
- net Led: no longer names the net of D3.2 (A), R10.1
- net Led: no longer J3.1 (Pin_1)
Other:
- moved on the sheet: D3, R10

Commit message: Replace IRF740 by IRF530; Update PCB Layout; Plot PCB Layers
Parts:
- removed Q1, Q2: IRF740, Package_TO_SOT_THT:TO-220-3_Vertical, symbol Transistor_FET:IRF740
- added Q1, Q2: IRF530, Package_TO_SOT_THT:TO-220-3_Vertical, symbol SamacSys_Parts:IRF530
- R11: value (none) -> 10K
- R12: value (none) -> 100
- R13: value (none) -> 220
Connections:
- net GND: now also Q1.3, Q2.3
- net REDLeds: now also Q1.1
- net RED_Led_Array: now also Q1.2
- net UVLeds: now also Q2.1
- net UV_Led_Array: now also Q2.2
Other:
- moved on the sheet: D1, D2, D4, SW5
