File: Schematics/lightbox/8SegmentDisplay/8SegmentDisplay.kicad_sch (KiCad schematic)
At the start: 4 parts

Commit message: Fix annotations
Parts:
- renumbered J4 to J5
Changed lines of the file:
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@@
   (symbol (lib_id "Connector:Conn_01x11_Male") (at 106.68 97.79 0) (mirror y) (unit 1)
     (in_bom yes) (on_board yes)
-    (property "Reference" "J4" (id 0) (at 87.63 78.74 0)
+    (property "Reference" "J5" (id 0) (at 87.63 78.74 0)
       (effects (font (size 1.27 1.27)) (justify right))
     )

Commit message: Update lightbox design
Parts:
- J5: value ~ -> Conn_01x11_Pin; footprint Connector_PinHeader_1.27mm:PinHeader_1x12_P1.27mm_Vertical -> Connector_PinHeader_2.54mm:PinHeader_1x12_P2.54mm_Horizontal; symbol Connector:Conn_01x11_Male -> Connector:Conn_01x11_Pin
- U5, U6, U7: value ~ -> D148K
